Commit message: Add complete car urdf

File: complete_car/urdf/complete_car.urdf (robot description, URDF)
Before this commit: robot complete_car, 1 links, 0 joints
Links:
- removed link base_link
- added link body_car_chassis, mass 6.95519132903594; collision mesh filename=package://complete_car/meshes/body_car_chassis.STL; visual mesh filename=package://complete_car/meshes/body_car_chassis.STL
- added link body_car_wheel_left, mass 1.55682391481766; collision mesh filename=package://complete_car/meshes/body_car_wheel_left.STL; visual mesh filename=package://complete_car/meshes/body_car_wheel_left.STL
- added link body_car_wheel_right, mass 1.55682350721719; collision mesh filename=package://complete_car/meshes/body_car_wheel_right.STL; visual mesh filename=package://complete_car/meshes/body_car_wheel_right.STL
- added link head_car_chassis, mass 9.9942816842311; collision mesh filename=package://complete_car/meshes/head_car_chassis.STL; visual mesh filename=package://complete_car/meshes/head_car_chassis.STL
- added link head_car_wheel_left, mass 1.55682391481784; collision mesh filename=package://complete_car/meshes/head_car_wheel_left.STL; visual mesh filename=package://complete_car/meshes/head_car_wheel_left.STL
- added link head_car_wheel_right, mass 1.55682350721721; collision mesh filename=package://complete_car/meshes/head_car_wheel_right.STL; visual mesh filename=package://complete_car/meshes/head_car_wheel_right.STL
- added link spm1_base, mass 0.383954508133489; collision mesh filename=package://complete_car/meshes/spm1_base.STL; visual mesh filename=package://complete_car/meshes/spm1_base.STL
- added link spm1_leg1_distal, mass 0.0249434138951248; collision mesh filename=package://complete_car/meshes/spm1_leg1_distal.STL; visual mesh filename=package://complete_car/meshes/spm1_leg1_distal.STL
- added link spm1_leg1_platform, mass 0.0449010465380492; collision mesh filename=package://complete_car/meshes/spm1_leg1_platform.STL; visual mesh filename=package://complete_car/meshes/spm1_leg1_platform.STL
- added link spm1_leg1_proximal, mass 0.0687465305096129; collision mesh filename=package://complete_car/meshes/spm1_leg1_proximal.STL; visual mesh filename=package://complete_car/meshes/spm1_leg1_proximal.STL
- added link spm1_leg2_distal, mass 0.0249434660620519; collision mesh filename=package://complete_car/meshes/spm1_leg2_distal.STL; visual mesh filename=package://complete_car/meshes/spm1_leg2_distal.STL
- added link spm1_leg2_proximal, mass 0.0687464361626338; collision mesh filename=package://complete_car/meshes/spm1_leg2_proximal.STL; visual mesh filename=package://complete_car/meshes/spm1_leg2_proximal.STL
- added link spm1_leg3_distal, mass 0.0249434008867255; collision mesh filename=package://complete_car/meshes/spm1_leg3_distal.STL; visual mesh filename=package://complete_car/meshes/spm1_leg3_distal.STL
- added link spm1_leg3_proximal, mass 0.0687463808037662; collision mesh filename=package://complete_car/meshes/spm1_leg3_proximal.STL; visual mesh filename=package://complete_car/meshes/spm1_leg3_proximal.STL
- added link spm2_base, mass 0.383954508133489; collision mesh filename=package://complete_car/meshes/spm2_base.STL; visual mesh filename=package://complete_car/meshes/spm2_base.STL
- added link spm2_leg1_distal, mass 0.0249434138951242; collision mesh filename=package://complete_car/meshes/spm2_leg1_distal.STL; visual mesh filename=package://complete_car/meshes/spm2_leg1_distal.STL
- added link spm2_leg1_platform, mass 0.044901046538049; collision mesh filename=package://complete_car/meshes/spm2_leg1_platform.STL; visual mesh filename=package://complete_car/meshes/spm2_leg1_platform.STL
- added link spm2_leg1_proximal, mass 0.0687465305096126; collision mesh filename=package://complete_car/meshes/spm2_leg1_proximal.STL; visual mesh filename=package://complete_car/meshes/spm2_leg1_proximal.STL
- added link spm2_leg2_distal, mass 0.0249434660620516; collision mesh filename=package://complete_car/meshes/spm2_leg2_distal.STL; visual mesh filename=package://complete_car/meshes/spm2_leg2_distal.STL
- added link spm2_leg2_proximal, mass 0.0687464361626351; collision mesh filename=package://complete_car/meshes/spm2_leg2_proximal.STL; visual mesh filename=package://complete_car/meshes/spm2_leg2_proximal.STL
- added link spm2_leg3_distal, mass 0.0249434008867258; collision mesh filename=package://complete_car/meshes/spm2_leg3_distal.STL; visual mesh filename=package://complete_car/meshes/spm2_leg3_distal.STL
- added link spm2_leg3_proximal, mass 0.0687463808037651; collision mesh filename=package://complete_car/meshes/spm2_leg3_proximal.STL; visual mesh filename=package://complete_car/meshes/spm2_leg3_proximal.STL
- added link tail_car_chassis, mass 9.99428166268263; collision mesh filename=package://complete_car/meshes/tail_car_chassis.STL; visual mesh filename=package://complete_car/meshes/tail_car_chassis.STL
- added link tail_car_wheel_left, mass 1.55682391481766; collision mesh filename=package://complete_car/meshes/tail_car_wheel_left.STL; visual mesh filename=package://complete_car/meshes/tail_car_wheel_left.STL
- added link tail_car_wheel_right, mass 1.5568235072174; collision mesh filename=package://complete_car/meshes/tail_car_wheel_right.STL; visual mesh filename=package://complete_car/meshes/tail_car_wheel_right.STL
Joints:
- added joint body_car_wheel_left_joint: type continuous, parent body_car_chassis, child body_car_wheel_left, origin xyz=0 0.26953 0.0450000000000001 rpy=-1.5707963267949 0 0, axis 0 0 1
- added joint body_car_wheel_right_joint: type continuous, parent body_car_chassis, child body_car_wheel_right, origin xyz=0 -0.26869 0.0450000000000001 rpy=-1.5707963267949 0 0, axis 0 0 -1
- added joint head_car_chassis_joint: type fixed, parent spm1_leg1_platform, child head_car_chassis, origin xyz=-0.0116427344100918 -0.0116427344100924 0.0438572655899086 rpy=1.04516567956673 0.615479708670435 -2.35619449019237, axis 0 0 0
- added joint head_car_wheel_left_joint: type continuous, parent head_car_chassis, child head_car_wheel_left, origin xyz=0.276488513878161 0.269530000848736 -0.0369999949337831 rpy=-1.5707963267949 0 0, axis 0 0 1
- added joint head_car_wheel_right_joint: type continuous, parent head_car_chassis, child head_car_wheel_right, origin xyz=0.276488513878161 -0.269529999151265 -0.0369999949337831 rpy=-1.5707963267949 0 0, axis 0 0 -1
- added joint spm1_base_joint: type fixed, parent body_car_chassis, child spm1_base, origin xyz=0.18 0 0.0820210428191438 rpy=0 0 0, axis 0 0 0
- added joint spm1_leg1_base_proximal_joint: type revolute, parent spm1_base, child spm1_leg1_proximal, origin xyz=0.0372072256031851 -0.0479064844253887 0.0276377788636364 rpy=-2.03444393579569 0.420534335283973 -0.886077123792616, axis 0 0 -1, limit lower=0 upper=0 effort=0 velocity=0
- added joint spm1_leg1_distal_platform_joint: type revolute, parent spm1_leg1_distal, child spm1_leg1_platform, origin xyz=0.0555 0 0.0515000000000002 rpy=3.14159265358979 1.5707963267949 0, axis 0 0 1, limit lower=0 upper=0 effort=0 velocity=0
- added joint spm1_leg1_intermediate_distal_joint: type revolute, parent spm1_leg1_proximal, child spm1_leg1_distal, origin xyz=0 0.0515 0.06775 rpy=1.5707963267949 0 0, axis 0 0 1, limit lower=0 upper=0 effort=0 velocity=0
- added joint spm1_leg2_base_proximal_joint: type revolute, parent spm1_base, child spm1_leg2_proximal, origin xyz=0.0372072256031853 0 -0.0553386861731434 rpy=0.463647609000806 0.420534335283964 0.886077123792613, axis 0 0 -1, limit lower=0 upper=0 effort=0 velocity=0
- added joint spm1_leg2_intermediate_distal: type revolute, parent spm1_leg2_proximal, child spm1_leg2_distal, origin xyz=0 0.0515 0.06775 rpy=1.5707963267949 0 0, axis 0 0 1, limit lower=0 upper=0 effort=0 velocity=0
- added joint spm1_leg3_base_proximal: type revolute, parent spm1_base, child spm1_leg3_proximal, origin xyz=0.0372072256031854 0.0479064844253887 0.027637778863637 rpy=2.35619449019235 -0.955316618124513 0, axis 0 0 -1, limit lower=0 upper=0 effort=0 velocity=0
- added joint spm1_leg3_intermediate_distal: type revolute, parent spm1_leg3_proximal, child spm1_leg3_distal, origin xyz=0 0.0515 0.06775 rpy=1.5707963267949 0 0, axis 0 0 1, limit lower=0 upper=0 effort=0 velocity=0
- added joint spm2_base_joint: type fixed, parent body_car_chassis, child spm2_base, origin xyz=-0.18 0 0.0820210428191438 rpy=0 0 0, axis 0 0 0
- added joint spm2_leg1_base_proximal_joint: type revolute, parent spm2_base, child spm2_leg1_proximal, origin xyz=-0.0372072256031851 0.0479064844253887 0.0276377788636364 rpy=-2.0344439357957 0.420534335283973 2.25551552979718, axis 0 0 -1, limit lower=0 upper=0 effort=0 velocity=0
- added joint spm2_leg1_distal_platform: type revolute, parent spm2_leg1_distal, child spm2_leg1_platform, origin xyz=0.0555 0 0.0515000000000003 rpy=1.5707963267949 0 -1.5707963267949, axis 0 0 1, limit lower=0 upper=0 effort=0 velocity=0
- added joint spm2_leg1_intermediate_distal_joint: type revolute, parent spm2_leg1_proximal, child spm2_leg1_distal, origin xyz=0 0.0515 0.06775 rpy=1.5707963267949 0 0, axis 0 0 1, limit lower=0 upper=0 effort=0 velocity=0
- added joint spm2_leg2_base_proximal: type revolute, parent spm2_base, child spm2_leg2_proximal, origin xyz=-0.0372072256031853 0 -0.0553386861731434 rpy=0.463647609000806 0.420534335283964 -2.25551552979718, axis 0 0 -1, limit lower=0 upper=0 effort=0 velocity=0
- added joint spm2_leg2_intermediate_distal: type revolute, parent spm2_leg2_proximal, child spm2_leg2_distal, origin xyz=0 0.0515 0.06775 rpy=1.5707963267949 0 0, axis 0 0 1, limit lower=0 upper=0 effort=0 velocity=0
- added joint spm2_leg3_base_proximal_joint: type revolute, parent spm2_base, child spm2_leg3_proximal, origin xyz=-0.0372072256031855 -0.0479064844253887 0.027637778863637 rpy=2.35619449019235 -0.955316618124513 3.14159265358978, axis 0 0 -1, limit lower=0 upper=0 effort=0 velocity=0
- added joint spm2_leg3_intermediate_distal: type revolute, parent spm2_leg3_proximal, child spm2_leg3_distal, origin xyz=0 0.0514999999999999 0.0677499999999999 rpy=1.5707963267949 0 0, axis 0 0 1, limit lower=0 upper=0 effort=0 velocity=0
- added joint tail_car_chassis_joint: type fixed, parent spm2_leg1_platform, child tail_car_chassis, origin xyz=-0.0116427344100924 0.0116427344100917 0.0438572655899086 rpy=-1.04719755119659 -0.615479708670383 -0.785398163397444, axis 0 0 0
- added joint tail_car_wheel_left_joint: type continuous, parent tail_car_chassis, child tail_car_wheel_left, origin xyz=-0.276488513878146 0.269604621962139 -0.0364522685746904 rpy=-1.56876445516506 0 0, axis 0 0 1
- added joint tail_car_wheel_right_joint: type continuous, parent tail_car_chassis, child tail_car_wheel_right, origin xyz=-0.276488513878177 -0.269454265283014 -0.0375475685418142 rpy=-1.56876445516506 0 0, axis 0 0 -1
